File: hardware/parking_sensor_node/parking_sensor_node.kicad_pcb (KiCad board)
At the start: 2 copper layers, 99.1 x 91.4 mm, 14 parts, among them J1 RS485_BUS, J2 HC-SR04, U1 NUCLEO64-F411RE, U2 MAX3485

Commit message: hardware: carrier PCB for fabrication
Parts:
- D1: value LED_KRGB -> LED_BGKR; footprint LED_THT:LED_D5.0mm-4_RGB -> ParkingSensor:LED_D5.0mm-4_RGB_BGKR
Connections:
- D1 pad 1: GND -> Net-(D1-BA)
- D1 pad 2: Net-(D1-RA) -> Net-(D1-GA)
- D1 pad 3: Net-(D1-GA) -> GND
- D1 pad 4: Net-(D1-BA) -> Net-(D1-RA)
Routing:
- net Net-(D1-GA): track 9.20 -> 17.5 mm
- net Net-(D1-BA): track 6.89 -> 10.5 mm
- net Net-(D1-RA): track 9.17 -> 6.89 mm
- net GND: track 58.3 -> 59.4 mm
Changed lines of the file:
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@@
 		(tenting front back)
 		(pcbplotparams
-			(layerselection 0x00000000_00000000_55555555_5755f5ff)
+			(layerselection 0x00000000_00000000_55555555_575555ff)
 			(plot_on_all_layers_selection 0x00000000_00000000_00000000_00000000)
 			(disableapertmacros no)
@@
 			(outputformat 1)
 			(mirror no)
-			(drillshape 1)
+			(drillshape 0)
 			(scaleselection 1)
-			(outputdirectory "")
+			(outputdirectory "gerber/")
 		)
 	)
@@
 		)
 	)
-	(footprint "LED_THT:LED_D5.0mm-4_RGB"
+	(footprint "ParkingSensor:LED_D5.0mm-4_RGB_BGKR"
 		(layer "F.Cu")
 		(at 266.07 40.64)
@@
 			)
 		)
-		(property "Value" "LED_KRGB"
+		(property "Value" "LED_BGKR"
 			(at 1.905 3.96 0)
 			(layer "F.Fab")
@@
 			)
 		)
-		(property "Description" "RGB LED, cathode/red/green/blue"
+		(property "Description" "RGB LED, blue/green/cathode/red"
 			(at 0 0 0)
 			(layer "F.Fab")
@@
 			(at 0 0)
 			(size 1.07 1.8)
-			(drill 0.9)
+			(drill 0.8)
 			(layers "*.Cu" "*.Mask")
 			(remove_unused_layers no)
-			(net 1 "GND")
-			(pinfunction "K")
+			(net 5 "Net-(D1-BA)")
+			(pinfunction "BA")
 			(pintype "passive")
 		)
@@
 			(at 1.27 0)
 			(size 1.07 1.8)
-			(drill 0.9)
+			(drill 0.8)
 			(layers "*.Cu" "*.Mask")
 			(remove_unused_layers no)
-			(net 4 "Net-(D1-RA)")
-			(pinfunction "RA")
+			(net 3 "Net-(D1-GA)")
+			(pinfunction "GA")
 			(pintype "passive")
 		)
@@
 			(at 2.54 0)
 			(size 1.07 1.8)
-			(drill 0.9)
+			(drill 0.8)
 			(layers "*.Cu" "*.Mask")
 			(remove_unused_layers no)
-			(net 3 "Net-(D1-GA)")
-			(pinfunction "GA")
+			(net 1 "GND")
+			(pinfunction "K")
 			(pintype "passive")
 		)
@@
 			(at 3.81 0)
 			(size 1.07 1.8)
-			(drill 0.9)
+			(drill 0.8)
 			(layers "*.Cu" "*.Mask")
 			(remove_unused_layers no)
-			(net 5 "Net-(D1-BA)")
-			(pinfunction "BA")
+			(net 4 "Net-(D1-RA)")
+			(pinfunction "RA")
 			(pintype "passive")
 		)
@@
 	)
 	(segment
-		(start 266.07 40.64)
-		(end 263.9 42.81)
+		(start 247.769 67.191)
+		(end 248.92 66.04)
 		(width 0.2)
 		(layer "F.Cu")
@@
 	)
 	(segment
-		(start 247.769 67.191)
-		(end 248.92 66.04)
+		(start 268.61 41.005)
+		(end 270.705 43.1)
 		(width 0.2)
 		(layer "F.Cu")
@@
 	)
 	(segment
+		(start 270.705 43.1)
+		(end 271.9 43.1)
+		(width 0.2)
+		(layer "F.Cu")
+		(net 1)
+	)
+	(segment
 		(start 251.46 79.41424)
 		(end 250.071 80.80324)
@@
 	)
 	(segment
+		(start 268.61 40.275)
+		(end 268.61 40.64)
+		(width 0.2)
+		(layer "F.Cu")
+		(net 1)
+	)
+	(segment
 		(start 251.46 78.74)
 		(end 251.46 79.41424)
@@
 	)
 	(segment
-		(start 263.9 42.81)
-		(end 263.9 43.4)
+		(start 268.61 40.64)
+		(end 268.61 41.005)
 		(width 0.2)
 		(layer "F.Cu")
@@
 	)
 	(segment
-		(start 263.9 43.4)
-		(end 263.9 43.5)
-		(width 0.2)
-		(layer "F.Cu")
-		(net 1)
-	)
-	(segment
 		(start 274.96 25.84)
 		(end 274.9 25.9)
@@
 	)
 	(via
-		(at 263.9 43.4)
+		(at 258.4 57.9)
 		(size 0.6)
 		(drill 0.3)
@@
 	)
 	(via
-		(at 258.4 57.9)
+		(at 274.9 25.9)
 		(size 0.6)
 		(drill 0.3)
@@
 	)
 	(via
-		(at 274.9 25.9)
+		(at 269.1 59.1)
 		(size 0.6)
 		(drill 0.3)
@@
 	)
 	(via
-		(at 269.1 59.1)
+		(at 276.5 30.5)
 		(size 0.6)
 		(drill 0.3)
@@
 	)
 	(via
-		(at 276.5 30.5)
+		(at 275.2 50.8)
 		(size 0.6)
 		(drill 0.3)
@@
 	)
 	(via
-		(at 275.2 50.8)
+		(at 271.9 43.1)
 		(size 0.6)
 		(drill 0.3)
@@
 	)
 	(segment
-		(start 268.61 40.275)
-		(end 268.61 40.64)
+		(start 268.176 39.439)
+		(end 267.34 40.275)
 		(width 0.2)
 		(layer "F.Cu")
@@
 	)
 	(segment
-		(start 274.245 40.64)
-		(end 274.245 39.195057)
+		(start 275.0585 39.8265)
+		(end 275.0585 34.87484)
 		(width 0.2)
 		(layer "F.Cu")
@@
 	)
 	(segment
-		(start 271.381 37.619)
-		(end 270.9 38.1)
+		(start 270.23766 39.439)
+		(end 268.176 39.439)
 		(width 0.2)
 		(layer "F.Cu")
@@
 	)
 	(segment
-		(start 270.9 38.1)
-		(end 270.785 38.1)
+		(start 273.4315 36.24516)
+		(end 270.23766 39.439)
 		(width 0.2)
 		(layer "F.Cu")
@@
 	)
 	(segment
-		(start 274.245 39.195057)
-		(end 272.668943 37.619)
+		(start 267.34 40.275)
+		(end 267.34 40.64)
 		(width 0.2)
 		(layer "F.Cu")
@@
 	)
 	(segment
-		(start 270.785 38.1)
-		(end 268.61 40.275)
+		(start 273.4315 34.87484)
+		(end 273.4315 36.24516)
 		(width 0.2)
 		(layer "F.Cu")
@@
 	)
 	(segment
-		(start 272.668943 37.619)
-		(end 271.381 37.619)
+		(start 275.0585 34.87484)
+		(end 274.74266 34.559)
 		(width 0.2)
 		(layer "F.Cu")
@@
 	)
 	(segment
-		(start 267.34 40.362717)
-		(end 271.141717 36.561)
+		(start 274.74266 34.559)
+		(end 273.74734 34.559)
 		(width 0.2)
 		(layer "F.Cu")
-		(net 4)
+		(net 3)
 	)
 	(segment
-		(start 267.34 40.64)
-		(end 267.34 40.362717)
+		(start 274.245 40.64)
+		(end 275.0585 39.8265)
 		(width 0.2)
 		(layer "F.Cu")
-		(net 4)
+		(net 3)
 	)
 	(segment
-		(start 271.141717 36.561)
-		(end 273.244 36.561)
+		(start 273.74734 34.559)
+		(end 273.4315 34.87484)
+		(width 0.2)
+		(layer "F.Cu")
+		(net 3)
+	)
+	(segment
+		(start 274.245 36.275)
+		(end 269.88 40.64)
 		(width 0.2)
 		(layer "F.Cu")
@@
 	)
 	(segment
-		(start 273.244 36.561)
-		(end 274.245 35.56)
+		(start 274.245 35.56)
+		(end 274.245 36.275)
 		(width 0.2)
 		(layer "F.Cu")
@@
 	)
 	(segment
-		(start 269.88 40.64)
-		(end 274.245 45.005)
+		(start 273.225 44.7)
+		(end 269.765 44.7)
+		(width 0.2)
+		(layer "F.Cu")
+		(net 5)
+	)
+	(segment
+		(start 269.765 44.7)
+		(end 266.07 41.005)
+		(width 0.2)
+		(layer "F.Cu")
+		(net 5)
+	)
+	(segment
+		(start 266.07 41.005)
+		(end 266.07 40.64)
 		(width 0.2)
 		(layer "F.Cu")
@@
 	)
 	(segment
-		(start 274.245 45.005)
-		(end 274.245 45.72)
+		(start 274.245 45.72)
+		(end 273.225 44.7)
 		(width 0.2)
 		(layer "F.Cu")
