File: hardware/parking_sensor_node/parking_sensor_node.kicad_sch (KiCad schematic)
At the start: 14 parts, among them J1 RS485_BUS, J2 HC-SR04, U1 NUCLEO64-F411RE, U2 MAX3485

Commit message: hardware: carrier PCB for fabrication
Parts:
- D1: value LED_KRGB -> LED_BGKR; footprint LED_THT:LED_D5.0mm-4_RGB -> ParkingSensor:LED_D5.0mm-4_RGB_BGKR; symbol Device:LED_KRGB -> Device:LED_BGKR
Connections:
- net GND: now also D1.3 (K); no longer D1.1 (K)
- net at R5.2: now also D1.4 (RA); no longer D1.2 (RA)
- net at R6.2: now also D1.2 (GA); no longer D1.3 (GA)
- net at R7.2: now also D1.1 (BA); no longer D1.4 (BA)
Changed lines of the file:
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@@
 	)
 	(symbol
-		(lib_id "Device:LED_KRGB")
+		(lib_id "Device:LED_BGKR")
 		(at 171.45 116.84 0)
 		(mirror y)
@@
 			)
 		)
-		(property "Value" "LED_KRGB"
+		(property "Value" "LED_BGKR"
 			(at 171.45 105.41 0)
 			(effects
@@
 			)
 		)
-		(property "Footprint" "LED_THT:LED_D5.0mm-4_RGB"
+		(property "Footprint" "ParkingSensor:LED_D5.0mm-4_RGB_BGKR"
 			(at 171.45 118.11 0)
 			(effects
@@
 			)
 		)
-		(property "Description" "RGB LED, cathode/red/green/blue"
+		(property "Description" "RGB LED, blue/green/cathode/red"
 			(at 171.45 116.84 0)
 			(effects
